File: layouts/default/default.kicad_pcb (KiCad board)
At the start: 2 copper layers, 0 parts

Commit message: built
Parts:
- added C1: 100nF ±10% 16V X7R, atopile:C0402-b3ef17, F.Cu at (50.0, -50.0)
- added C10: 100nF ±10% 16V X7R, atopile:C0402-b3ef17, F.Cu at (60.0, 0.00)
- added C11: 10µF ±10% 25V X5R, atopile:C0805-3b2e55, F.Cu at (20.0, -20.0)
- added C12: 10µF ±10% 25V X5R, atopile:C0805-3b2e55, F.Cu at (20.0, -10.0)
- added C13: 100nF ±10% 16V X7R, atopile:C0402-b3ef17, F.Cu at (20.0, 0.00)
- added C2: 100nF ±10% 16V X7R, atopile:C0402-b3ef17, F.Cu at (50.0, 0.00)
- added C3: 100nF ±10% 16V X7R, atopile:C0402-b3ef17, F.Cu at (50.0, -110.0)
- added C4: 100nF ±10% 16V X7R, atopile:C0402-b3ef17, F.Cu at (50.0, -180.0)
- added C5: 100nF ±10% 16V X7R, atopile:C0402-b3ef17, F.Cu at (50.0, -60.0)
- added C6: 100nF ±10% 16V X7R, atopile:C0402-b3ef17, F.Cu at (50.0, -20.0)
- added C7: 100nF ±10% 16V X7R, atopile:C0402-b3ef17, F.Cu at (50.0, -70.0)
- added C8: 100nF ±10% 16V X7R, atopile:C0402-b3ef17, F.Cu at (50.0, -10.0)
- added C9: 100nF ±10% 50V X7R, atopile:C0805-3b2e55, F.Cu at (60.0, -10.0)
- added D1: , atopile:SOD-123F_L2.7-W1.6-LS3.8-RD-1-139753, F.Cu at (10.0, -210.0)
- added F1: , atopile:F0603-5fdc66, F.Cu at (10.0, -180.0)
- added LED1: , atopile:SENSOR-TH_BPW34-c0a4b0, F.Cu at (50.0, -140.0)
- added LED2: , atopile:SENSOR-TH_BPW34-c0a4b0, F.Cu at (50.0, -100.0)
- added LED3: , atopile:SENSOR-TH_BPW34-c0a4b0, F.Cu at (50.0, -210.0)
- added LED4: , atopile:SENSOR-TH_BPW34-c0a4b0, F.Cu at (50.0, -170.0)
- added R1: 0Ω 50mW, atopile:R0201-27027e, F.Cu at (50.0, -190.0)
- added R10: 1kΩ ±1% 62.5mW, atopile:R0402-56259e, F.Cu at (60.0, -40.0)
- added R11: 1kΩ ±1% 62.5mW, atopile:R0402-56259e, F.Cu at (60.0, -20.0)
- added R12: 10kΩ ±1% 62.5mW, atopile:R0402-56259e, F.Cu at (30.0, 0.00)
- added R2: 0Ω 50mW, atopile:R0201-27027e, F.Cu at (50.0, -150.0)
- added R3: 0Ω 50mW, atopile:R0201-27027e, F.Cu at (50.0, -120.0)
- added R4: 0Ω 50mW, atopile:R0201-27027e, F.Cu at (50.0, -80.0)
- added R5: 0Ω 50mW, atopile:R0201-27027e, F.Cu at (50.0, -160.0)
- added R6: 0Ω 50mW, atopile:R0201-27027e, F.Cu at (50.0, -90.0)
- added R7: 0Ω 50mW, atopile:R0201-27027e, F.Cu at (50.0, -30.0)
- added R8: 10kΩ ±1% 100mW, atopile:R0603-ebcab9, F.Cu at (50.0, -40.0)
- added R9: 0Ω 50mW, atopile:R0201-27027e, F.Cu at (50.0, -130.0)
- added U1: , atopile:SOIC-8_L5.0-W4.0-P1.27-LS6.0-BL-294f77, F.Cu at (50.0, -200.0)
- added U10: 1nF ±20% 50V X7R, atopile:C0402-b3ef17, F.Cu at (10.0, -130.0)
- added U11: , lib:SOT-23-6_L2.9-W1.6-P0.95-LS2.8-BR, F.Cu at (10.0, -60.0)
- added U12: 1MΩ ±1% 62.5mW, atopile:R0402-56259e, F.Cu at (10.0, -100.0)
- added U13: 450kΩ ±1% 62.5mW, atopile:R0402-56259e, F.Cu at (10.0, -140.0)
- added U14: 1kΩ ±1% 62.5mW, atopile:R0402-56259e, F.Cu at (10.0, 0.00)
- added U15: 100Ω ±1% 62.5mW, atopile:R0402-56259e, F.Cu at (10.0, -160.0)
- added U16: 1kΩ ±1% 62.5mW, atopile:R0402-56259e, F.Cu at (10.0, -110.0)
- added U17: 1kΩ ±1% 62.5mW, atopile:R0402-56259e, F.Cu at (10.0, -10.0)
- added U18: 10mΩ ±1% 1W, atopile:R1206-bdb864, F.Cu at (10.0, -40.0)
- added U19: , lib:IND-SMD_L6.6-W6.4, F.Cu at (10.0, -120.0)
- added U2: , atopile:GPSM-SMD_ATGM336H-TR-d79f58, F.Cu at (0.00, 0.00)
- added U20: , lib:CONN-TH_B2B-PH-K-S, F.Cu at (10.0, -170.0)
- added U21: , lib:CONN-TH_B2B-PH-K-S, F.Cu at (10.0, -80.0)
- added U22: , lib:CONN-TH_B2B-PH-K-S, F.Cu at (10.0, -150.0)
- added U23: , atopile:SOT-23-3_L2.9-W1.3-P1.90-LS2.4-BR-688f29, F.Cu at (10.0, -220.0)
- added U24: , lib:TSSOP-8_L4.4-W3.0-P0.65-LS6.4-BL, F.Cu at (10.0, -20.0)
- added U25: , lib:KEY-SMD_4P-L4.2-W3.2-P2.20-LS4.6, F.Cu at (40.0, 0.00)
- added U26: , lib:WIRELM-SMD_ESP32-S3-WROOM-1, F.Cu at (20.0, -30.0)
- added U3: , atopile:WIRELM-SMD_E22-900M30S-98c301, F.Cu at (60.0, -30.0)
- added U4: 100nF ±10% 16V X7R, atopile:C0402-b3ef17, F.Cu at (10.0, -50.0)
- added U5: 1µF ±10% 25V X5R, atopile:C0402-b3ef17, F.Cu at (10.0, -30.0)
- added U6: 10µF ±10% 10V X5R, atopile:C0603-bd72f6, F.Cu at (10.0, -90.0)
- added U7: 100nF ±10% 16V X7R, atopile:C0402-b3ef17, F.Cu at (10.0, -200.0)
- added U8: 4.7µF ±10% 10V X5R, atopile:C0603-bd72f6, F.Cu at (10.0, -190.0)
- added U9: 10µF ±10% 10V X5R, atopile:C0603-bd72f6, F.Cu at (10.0, -70.0)
